File: Backplane.kicad_pcb (KiCad board)
At the start: 4 copper layers, 167.6 x 96.5 mm, 59 parts, among them J1 Bus_PCI_Express_x16, U1 LTC3810IG_PBF, U2 ADP7104ACPZ-3.0-R7, U3 ISP817CXSM, U4 ISP817CXSM, U5 ISP817CXSM, U6 ISP817CXSM, U7 ISP817CXSM, U8 ISP817CXSM

Commit message: Merged both -1/-2 and backplane
Parts:
- removed D13, D14: MBR745, Package_TO_SOT_THT:TO-220-2_Vertical
- removed MOSFET1, MOSFET2, MOSFET3: SI7850DP-T1-E3, SDII Lib:POWERPAK_SO-8_SINGLE_VIS
- added C10: 10u, Capacitor_SMD:C_1206_3216Metric, F.Cu at (226.6, 111.9)
- added C11: 10u, Capacitor_SMD:C_1206_3216Metric, F.Cu at (224.2, 59.3)
- added C12: 10u, Capacitor_SMD:C_1206_3216Metric, F.Cu at (234.7, 100.2)
- added C13: 10u, Capacitor_SMD:C_1206_3216Metric, F.Cu at (236.7, 70.3)
- added C14: 10u, Capacitor_SMD:C_1206_3216Metric, B.Cu at (223.8, 65.7)
- added C15: 10u, Capacitor_SMD:C_1206_3216Metric, B.Cu at (222.8, 102.7)
- added C16: 10u, Capacitor_SMD:C_1206_3216Metric, B.Cu at (208.8, 54.1)
- added C17: 10u, Capacitor_SMD:C_1206_3216Metric, B.Cu at (214.2, 115.7)
- added C18: 10u, Capacitor_SMD:C_1206_3216Metric, B.Cu at (189.3, 57.1)
- added C19: 10u, Capacitor_SMD:C_1206_3216Metric, B.Cu at (194.0, 115.7)
- added C20: 10u, Capacitor_SMD:C_1206_3216Metric, B.Cu at (161.0, 76.8)
- added C21: 10u, Capacitor_SMD:C_1206_3216Metric, B.Cu at (161.5, 81.4)
- added C22: 10u, Capacitor_SMD:C_1206_3216Metric, B.Cu at (180.6, 71.3)
- added C23: 10u, Capacitor_SMD:C_1206_3216Metric, B.Cu at (173.5, 99.9)
- added C9: 10u, Capacitor_SMD:C_1206_3216Metric, F.Cu at (205.1, 56.4)
- added CR1: SMDJ85A, SDII Lib:SMDJ85A, B.Cu at (197.0, 95.9)
- added CR10: SMDJ33A, SDII Lib:SMDJ33A, F.Cu at (199.6, 75.5)
- added CR12: SMDJ33A, SDII Lib:SMDJ33A, F.Cu at (218.0, 87.9)
- added CR14: SMDJ33A, SDII Lib:SMDJ33A, F.Cu at (210.0, 95.4)
- added CR16: SMDJ33A, SDII Lib:SMDJ33A, F.Cu at (215.0, 80.9)
- added CR18: SMDJ33A, SDII Lib:SMDJ33A, B.Cu at (204.0, 95.9)
- added CR19: SMDJ33A, SDII Lib:SMDJ33A, B.Cu at (199.6, 75.4)
- added CR20: SMDJ33A, SDII Lib:SMDJ33A, B.Cu at (211.3, 97.4)
- added CR24: SMDJ33A, SDII Lib:SMDJ33A, B.Cu at (206.9, 75.5)
- added CR25: SMDJ33A, SDII Lib:SMDJ33A, B.Cu at (219.5, 87.9)
- added CR26: SMDJ33A, SDII Lib:SMDJ33A, B.Cu at (215.0, 80.9)
- added CR27: SMDJ6.0A, SDII Lib:SMDJ6_0A, F.Cu at (162.5, 85.4)
- added CR28: SMDJ6.0A, SDII Lib:SMDJ6_0A, F.Cu at (169.0, 77.4)
- added CR29: SMDJ6.0A, SDII Lib:SMDJ6_0A, F.Cu at (169.0, 93.5)
- added CR30: SMDJ6.0A, SDII Lib:SMDJ6_0A, F.Cu at (176.5, 77.4)
- added CR31: SMDJ6.0A, SDII Lib:SMDJ6_0A, F.Cu at (176.5, 93.4)
- added CR32: RF201LAM2STR, SDII Lib:RF201LAM2STR(new_POW_diode), F.Cu at (197.0, 95.9)
- added CR33: RBR1MM60ATFTR, SDII Lib:RBR1MM60ATFTR(new_VR_diode), F.Cu at (202.0, 101.9)
- added CR34: RBR1MM60ATFTR, SDII Lib:RBR1MM60ATFTR(new_VR_diode), F.Cu at (198.5, 69.4)
- added CR35: RBR1MM60ATFTR, SDII Lib:RBR1MM60ATFTR(new_VR_diode), F.Cu at (209.0, 101.4)
- added CR36: RBR1MM60ATFTR, SDII Lib:RBR1MM60ATFTR(new_VR_diode), F.Cu at (205.7, 69.7)
- added CR37: RBR1MM60ATFTR, SDII Lib:RBR1MM60ATFTR(new_VR_diode), F.Cu at (216.1, 92.6)
- added CR38: RBR1MM60ATFTR, SDII Lib:RBR1MM60ATFTR(new_VR_diode), F.Cu at (213.2, 76.2)
- added CR39: RBR1MM60ATFTR, SDII Lib:RBR1MM60ATFTR(new_VR_diode), B.Cu at (202.0, 101.9)
- added CR40: RBR1MM60ATFTR, SDII Lib:RBR1MM60ATFTR(new_VR_diode), B.Cu at (198.5, 69.4)
- added CR41: RBR1MM60ATFTR, SDII Lib:RBR1MM60ATFTR(new_VR_diode), B.Cu at (209.0, 103.9)
- added CR42: RBR1MM60ATFTR, SDII Lib:RBR1MM60ATFTR(new_VR_diode), B.Cu at (205.7, 69.7)
- added CR43: RBR1MM60ATFTR, SDII Lib:RBR1MM60ATFTR(new_VR_diode), B.Cu at (217.6, 92.6)
- added CR44: RBR1MM60ATFTR, SDII Lib:RBR1MM60ATFTR(new_VR_diode), B.Cu at (213.2, 76.2)
- added CR6: SMDJ33A, SDII Lib:SMDJ33A, F.Cu at (203.0, 95.9)
- added CR8: SMDJ33A, SDII Lib:SMDJ33A, F.Cu at (206.9, 75.5)
- added D27: 1N5819HW-7-F, SDII Lib:1N5819, B.Cu at (156.5, 81.4)
- added D28: 1N5819HW-7-F, SDII Lib:1N5819, B.Cu at (155.5, 86.1)
- added D29: 1N5819HW-7-F, SDII Lib:1N5819, B.Cu at (171.0, 73.1)
- added D30: 1N5819HW-7-F, SDII Lib:1N5819, B.Cu at (166.0, 72.0)
- added D31: 1N5819HW-7-F, SDII Lib:1N5819, B.Cu at (161.5, 98.3)
- added D32: 1N5819HW-7-F, SDII Lib:1N5819, B.Cu at (166.5, 99.3)
- added D33: 1N5819HW-7-F, SDII Lib:1N5819, B.Cu at (175.5, 71.4)
- added D34: 1N5819HW-7-F, SDII Lib:1N5819, B.Cu at (174.5, 76.4)
- added D35: 1N5819HW-7-F, SDII Lib:1N5819, B.Cu at (178.5, 99.8)
- added D36: 1N5819HW-7-F, SDII Lib:1N5819, B.Cu at (179.5, 95.4)
- added D37: SMDJ60CA, SDII Lib:SMDJ6_0CA, F.Cu at (183.7, 74.9)
- added D38: SMDJ60CA, SDII Lib:SMDJ6_0CA, F.Cu at (183.5, 95.8)
- added D39: SMDJ60CA, SDII Lib:SMDJ6_0CA, B.Cu at (188.1, 74.9)
- added D40: SMDJ60CA, SDII Lib:SMDJ6_0CA, B.Cu at (187.9, 95.8)
- added D41: SMDJ60CA, SDII Lib:SMDJ6_0CA, F.Cu at (192.7, 74.8)
- added D42: SMDJ60CA, SDII Lib:SMDJ6_0CA, F.Cu at (192.3, 95.9)
- added H1: MountingHole, MountingHole:MountingHole_3.2mm_M3, F.Cu at (157.5, 48.0)
- added H2: MountingHole, MountingHole:MountingHole_3.2mm_M3, F.Cu at (333.0, 47.5)
- added H3: MountingHole, MountingHole:MountingHole_3.2mm_M3, F.Cu at (333.0, 134.5)
- added H4: MountingHole, MountingHole:MountingHole_3.2mm_M3, F.Cu at (157.0, 135.0)
- added J2: 10018783-10202TLF, SDII Lib:PCI_Express_Card, F.Cu at (276.8, 103.3)
- added J3: 10018783-10202TLF, SDII Lib:PCI_Express_Card, F.Cu at (292.8, 103.3)
- added J4: 10018783-10202TLF, SDII Lib:PCI_Express_Card, F.Cu at (308.8, 103.3)
- added J5: 10018783-10202TLF, SDII Lib:PCI_Express_Card, F.Cu at (324.8, 103.3)
- added J6: 5019514000, SDII Lib:BP_Connector, F.Cu at (192.7, 86.0)
- added R100: 1k, Resistor_SMD:R_0805_2012Metric, F.Cu at (319.0, 72.3)
- added R24: 15k, Resistor_SMD:R_0805_2012Metric, F.Cu at (159.6, 103.5)
- added R25: 4.7k, Resistor_SMD:R_0805_2012Metric, F.Cu at (161.9, 109.4)
- added R26: 3k, Resistor_SMD:R_0805_2012Metric, B.Cu at (208.5, 115.9)
- added R27: 1k, Resistor_SMD:R_0805_2012Metric, B.Cu at (194.3, 119.9)
- added R28: 3k, Resistor_SMD:R_0805_2012Metric, B.Cu at (203.6, 57.5)
- added R29: 1k, Resistor_SMD:R_0805_2012Metric, B.Cu at (189.5, 61.4)
- added R30: 3k, Resistor_SMD:R_0805_2012Metric, B.Cu at (228.5, 116.2)
- added R31: 1k, Resistor_SMD:R_0805_2012Metric, B.Cu at (214.5, 119.9)
- added R32: 3k, Resistor_SMD:R_0805_2012Metric, B.Cu at (223.0, 54.4)
- added R33: 1k, Resistor_SMD:R_0805_2012Metric, B.Cu at (209.0, 58.3)
- added R34: 3k, Resistor_SMD:R_0805_2012Metric, B.Cu at (237.0, 103.1)
- added R35: 1k, Resistor_SMD:R_0805_2012Metric, B.Cu at (223.0, 106.8)
- added R36: 3k, Resistor_SMD:R_0805_2012Metric, B.Cu at (238.0, 66.1)
- added R37: 1k, Resistor_SMD:R_0805_2012Metric, B.Cu at (223.9, 69.8)
- added R38: 1K, Resistor_SMD:R_0805_2012Metric, B.Cu at (205.5, 102.9)
- added R39: 1K, Resistor_SMD:R_0805_2012Metric, F.Cu at (205.5, 102.9)
- added R40: 1K, Resistor_SMD:R_0805_2012Metric, F.Cu at (209.3, 68.6)
- added R41: 1K, Resistor_SMD:R_0805_2012Metric, F.Cu at (202.0, 68.4)
- added R42: 1K, Resistor_SMD:R_0805_2012Metric, F.Cu at (220.5, 92.4)
- added R43: 1K, Resistor_SMD:R_0805_2012Metric, F.Cu at (212.5, 102.9)
- added R44: 1K, Resistor_SMD:R_0805_2012Metric, F.Cu at (217.5, 76.4)
- added R45: 1K, Resistor_SMD:R_0805_2012Metric, B.Cu at (202.0, 68.4)
- added R46: 1K, Resistor_SMD:R_0805_2012Metric, B.Cu at (213.0, 104.9)
- added R47: 1K, Resistor_SMD:R_0805_2012Metric, B.Cu at (209.3, 68.6)
- added R48: 1K, Resistor_SMD:R_0805_2012Metric, B.Cu at (223.0, 92.4)
- added R49: 1K, Resistor_SMD:R_0805_2012Metric, B.Cu at (217.5, 76.4)
- added R50: 100K, Resistor_SMD:R_0805_2012Metric, B.Cu at (157.9, 91.2)
- added R51: 100K, Resistor_SMD:R_0805_2012Metric, B.Cu at (170.8, 77.5)
- added R52: 100K, Resistor_SMD:R_0805_2012Metric, B.Cu at (171.4, 96.9)
- added R53: 100K, Resistor_SMD:R_0805_2012Metric, B.Cu at (177.0, 81.3)
- added R54: 100K, Resistor_SMD:R_0805_2012Metric, B.Cu at (177.1, 90.1)
- added R55: 10K, Resistor_SMD:R_0805_2012Metric, B.Cu at (183.7, 74.8)
- added R56: 10K, Resistor_SMD:R_0805_2012Metric, B.Cu at (183.5, 95.8)
- added R57: 10K, Resistor_SMD:R_0805_2012Metric, F.Cu at (188.1, 74.9)
- added R58: 10K, Resistor_SMD:R_0805_2012Metric, F.Cu at (187.9, 95.8)
- added R59: 10K, Resistor_SMD:R_0805_2012Metric, B.Cu at (192.5, 74.8)
- added R60: 10K, Resistor_SMD:R_0805_2012Metric, B.Cu at (192.5, 95.9)
- added R61: 2.2k, Resistor_SMD:R_0805_2012Metric, F.Cu at (241.7, 126.6)
- added R62: 200, Resistor_SMD:R_0402_1005Metric, F.Cu at (239.4, 126.7)
- added R63: 2.2k, Resistor_SMD:R_0805_2012Metric, F.Cu at (162.0, 102.8)
- added R64: 200, Resistor_SMD:R_0402_1005Metric, B.Cu at (162.5, 106.5)
- added R65: 200, Resistor_SMD:R_0402_1005Metric, F.Cu at (164.3, 109.4)
- added R66: 2, Resistor_SMD:R_0603_1608Metric, F.Cu at (245.2, 127.0)
- added R67: 2, Resistor_SMD:R_0603_1608Metric, F.Cu at (158.3, 109.5)
- added R68: 3k, Resistor_SMD:R_0805_2012Metric, F.Cu at (196.4, 108.2)
- added R69: 2k, Resistor_SMD:R_0805_2012Metric, F.Cu at (190.6, 58.1)
- added R70: 2k, Resistor_SMD:R_0805_2012Metric, F.Cu at (211.9, 114.2)
- added R71: 2k, Resistor_SMD:R_0805_2012Metric, F.Cu at (209.7, 61.0)
- added R72: 2k, Resistor_SMD:R_0805_2012Metric, F.Cu at (220.2, 101.9)
- added R73: 2k, Resistor_SMD:R_0805_2012Metric, F.Cu at (222.2, 72.2)
- added R74: 2k, Resistor_SMD:R_0805_2012Metric, B.Cu at (238.0, 69.5)
- added R75: 2k, Resistor_SMD:R_0805_2012Metric, B.Cu at (237.0, 106.6)
- added R76: 2k, Resistor_SMD:R_0805_2012Metric, B.Cu at (223.0, 57.8)
- added R77: 2k, Resistor_SMD:R_0805_2012Metric, B.Cu at (228.5, 119.7)
- added R78: 2k, Resistor_SMD:R_0805_2012Metric, B.Cu at (203.6, 61.0)
- added R79: 2k, Resistor_SMD:R_0805_2012Metric, B.Cu at (208.5, 119.4)
- added R80: 22k, Resistor_SMD:R_0805_2012Metric, B.Cu at (164.1, 135.7)
- added R81: 200k, Resistor_SMD:R_0805_2012Metric, F.Cu at (171.2, 134.1)
- added R82: 22k, Resistor_SMD:R_0805_2012Metric, B.Cu at (171.2, 134.2)
- added R83: 3k, Resistor_SMD:R_0805_2012Metric, F.Cu at (180.1, 130.9)
- added R84: 2k, Resistor_SMD:R_0805_2012Metric, F.Cu at (177.4, 132.1)
- added R85: 1.5k, Resistor_SMD:R_0805_2012Metric, F.Cu at (178.5, 134.1)
- added R86: 1k, Resistor_SMD:R_0805_2012Metric, F.Cu at (252.0, 71.0)
- added R87: 1k, Resistor_SMD:R_0805_2012Metric, F.Cu at (252.0, 66.4)
- added R88: 1k, Resistor_SMD:R_0805_2012Metric, F.Cu at (254.0, 62.5)
- added R89: 1k, Resistor_SMD:R_0805_2012Metric, F.Cu at (269.0, 77.5)
- added R90: 1k, Resistor_SMD:R_0805_2012Metric, F.Cu at (271.5, 73.5)
- added R92: 1k, Resistor_SMD:R_0805_2012Metric, F.Cu at (285.5, 77.6)
- added R94: 1k, Resistor_SMD:R_0805_2012Metric, F.Cu at (287.0, 73.4)
- added R95: 1k, Resistor_SMD:R_0805_2012Metric, F.Cu at (301.5, 77.5)
- added R99: 1k, Resistor_SMD:R_0805_2012Metric, F.Cu at (317.0, 76.0)
- added U10: ADP7104ACPZ-R7, SDII Lib:CP_8_5_ADI, F.Cu at (162.6, 106.5)
- added U11: ISP817CXSM, SDII Lib:ISP817SM_ISO, B.Cu at (201.5, 118.4)
- added U12: ISP817CXSM, SDII Lib:ISP817SM_ISO, B.Cu at (196.5, 59.9)
- added U13: ISP817CXSM, SDII Lib:ISP817SM_ISO, B.Cu at (221.5, 118.4)
- added U14: ISP817CXSM, SDII Lib:ISP817SM_ISO, B.Cu at (216.0, 56.9)
- added U15: ISP817CXSM, SDII Lib:ISP817SM_ISO, B.Cu at (230.0, 105.4)
- added U16: ISP817CXSM, SDII Lib:ISP817SM_ISO, B.Cu at (231.0, 68.4)
- added U17: OP191GSZ-REEL7, SDII Lib:OP191, B.Cu at (159.5, 86.4)
- added U18: OP191GSZ-REEL7, SDII Lib:OP191, B.Cu at (166.0, 76.0)
- added U19: OP191GSZ-REEL7, SDII Lib:OP191, B.Cu at (166.5, 95.3)
- added U20: OP191GSZ-REEL7, SDII Lib:OP191, B.Cu at (178.5, 76.4)
- added U21: OP191GSZ-REEL7, SDII Lib:OP191, B.Cu at (175.5, 94.9)
- added U9: ADP7104ACPZ-R7, SDII Lib:CP_8_5_ADI, F.Cu at (240.0, 132.0)
- C1: value 560p -> .47u; footprint Capacitor_THT:CP_Axial_L10.0mm_D4.5mm_P15.00mm_Horizontal -> Capacitor_SMD:C_0805_2012Metric
- C2: value .01u -> 0.1u; footprint Capacitor_THT:CP_Axial_L10.0mm_D4.5mm_P15.00mm_Horizontal -> Capacitor_SMD:C_0603_1608Metric
- C3: value 220p -> 3.3n; footprint Capacitor_THT:CP_Axial_L10.0mm_D4.5mm_P15.00mm_Horizontal -> Capacitor_SMD:C_0603_1608Metric
- C4: value 33p -> 33u; footprint Capacitor_THT:CP_Axial_L10.0mm_D4.5mm_P15.00mm_Horizontal -> Capacitor_SMD:C_1206_3216Metric
- C5: value 0.1u -> 22u; footprint Capacitor_THT:CP_Axial_L10.0mm_D4.5mm_P15.00mm_Horizontal -> Capacitor_SMD:C_1206_3216Metric
- C6: value 1u -> 22u; footprint Capacitor_THT:CP_Axial_L10.0mm_D4.5mm_P15.00mm_Horizontal -> Capacitor_SMD:C_1206_3216Metric
- C7: value 240u -> 10u; footprint Capacitor_THT:CP_Axial_L10.0mm_D4.5mm_P15.00mm_Horizontal -> Capacitor_SMD:C_1206_3216Metric; moved to B.Cu
- C8: value 2.2u -> 10u; footprint Capacitor_THT:CP_Axial_L10.0mm_D4.5mm_P15.00mm_Horizontal -> Capacitor_SMD:C_1206_3216Metric
- D1: value 1N4148 -> 1N5818; footprint Diode_THT:D_DO-35_SOD27_P7.62mm_Horizontal -> Diode_THT:D_DO-41_SOD81_P10.16mm_Horizontal
- D10, D11, D12, D3, D4, D5, D6, D7, D8, D9: value MBR745 -> 1N4148WS; footprint Package_TO_SOT_THT:TO-220-2_Vertical -> SDII Lib:1N4148WS
- D15: value 1N4007 -> 1N4148WS; footprint Diode_THT:D_DO-41_SOD81_P10.16mm_Horizontal -> SDII Lib:1N4148WS
- D2: value RB168MM100 -> 1N4148WS; footprint SDII Lib:SOD-123FL -> SDII Lib:1N4148WS
- J1: value Bus_PCI_Express_x16 -> 10018783-10202TLF; footprint Connector_PCBEdge:BUS_PCIexpress_x16 -> SDII Lib:PCI_Express_Card
- L1: value 7.6u -> 22u; footprint Inductor_SMD:L_Bourns_SRR1260 -> SDII Lib:IND_1210-WE-PD_WRE
- R1: value 10k -> 30k; footprint Resistor_THT:R_Axial_DIN0204_L3.6mm_D1.6mm_P5.08mm_Horizontal -> Resistor_SMD:R_0805_2012Metric
- R10: value 12 -> 100k; footprint Resistor_THT:R_Axial_DIN0204_L3.6mm_D1.6mm_P5.08mm_Horizontal -> Resistor_SMD:R_0805_2012Metric
- R11: value 100k -> 10; footprint Resistor_THT:R_Axial_DIN0204_L3.6mm_D1.6mm_P5.08mm_Horizontal -> Resistor_SMD:R_0805_2012Metric; moved to B.Cu
- R12: value 5k -> 2k; footprint Resistor_THT:R_Axial_DIN0204_L3.6mm_D1.6mm_P5.08mm_Horizontal -> Resistor_SMD:R_0805_2012Metric
- R13, R15, R17, R19, R21, R23: footprint Resistor_THT:R_Axial_DIN0204_L3.6mm_D1.6mm_P5.08mm_Horizontal -> Resistor_SMD:R_0805_2012Metric
- R14, R16, R18, R20, R22: value 5k -> 3k; footprint Resistor_THT:R_Axial_DIN0204_L3.6mm_D1.6mm_P5.08mm_Horizontal -> Resistor_SMD:R_0805_2012Metric
- R2: value 90.9k -> 20m; footprint Resistor_THT:R_Axial_DIN0204_L3.6mm_D1.6mm_P5.08mm_Horizontal -> Resistor_SMD:R_1206_3216Metric
- R3: value 100k -> 200k; footprint Resistor_THT:R_Axial_DIN0204_L3.6mm_D1.6mm_P5.08mm_Horizontal -> Resistor_SMD:R_0805_2012Metric
- R4: value 274k -> 30k; footprint Resistor_THT:R_Axial_DIN0204_L3.6mm_D1.6mm_P5.08mm_Horizontal -> Resistor_SMD:R_0805_2012Metric; moved to B.Cu
- R5: value 100k -> 10K; footprint Resistor_THT:R_Axial_DIN0204_L3.6mm_D1.6mm_P5.08mm_Horizontal -> Resistor_SMD:R_0805_2012Metric
- R6: value 8k -> 15k; footprint Resistor_THT:R_Axial_DIN0204_L3.6mm_D1.6mm_P5.08mm_Horizontal -> Resistor_SMD:R_0805_2012Metric
- R7: value 1k -> 10k; footprint Resistor_THT:R_Axial_DIN0204_L3.6mm_D1.6mm_P5.08mm_Horizontal -> Resistor_SMD:R_0805_2012Metric; moved to B.Cu
- R8: value 8k -> 100k; footprint Resistor_THT:R_Axial_DIN0204_L3.6mm_D1.6mm_P5.08mm_Horizontal -> Resistor_SMD:R_0805_2012Metric
- R9: value 1k -> 10; footprint Resistor_THT:R_Axial_DIN0204_L3.6mm_D1.6mm_P5.08mm_Horizontal -> Resistor_SMD:R_0805_2012Metric
- U1: value LTC3810IG_PBF -> LTC3894EFE-PBF; footprint SDII Lib:SSOP-28_G -> SDII Lib:TSSOP20-EP_4P4X6P5_ADI
- U2: value ADP7104ACPZ-3.0-R7 -> FDS4435A; footprint SDII Lib:CP_8_5_ADI -> SDII Lib:SOIC8_751EB_FAS
- moved J1 161.3 mm to (259.8, 103.3), turned to 90 degrees
- moved D15 159.8 mm to (200.0, 63.3)
- moved D4 157.5 mm to (215.9, 118.7)
- moved D3 152.8 mm to (203.9, 116.7)
- moved R13 127.5 mm to (208.4, 114.2), turned to 90 degrees
- moved U3 121.8 mm to (201.4, 112.7)
- moved R12 119.6 mm to (194.2, 111.3), turned to 90 degrees
- moved R1 113.1 mm to (177.4, 130.0)
- moved C5 108.0 mm to (247.5, 132.7), turned to 180 degrees
- moved C2 104.8 mm to (166.7, 131.6), turned to -90 degrees
- moved C1 103.7 mm to (177.0, 124.5), turned to -90 degrees
- moved U8 99.2 mm to (229.5, 72.9)
- moved U6 89.3 mm to (217.0, 61.9)
- moved U1 76.5 mm to (171.6, 127.4)
- moved R23 74.3 mm to (236.6, 74.4), turned to 90 degrees
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Connections:
- C1 pad 1: GND -> 28V_REF
- C1 pad 2: Net-(U1-SS/TRACK) -> Net-(U1-CAP)
- C2 pad 1: Net-(C2-Pad1) -> Net-(U1-TRACK/SS)
- C2 pad 2: Net-(U1-PL/LPF) -> GND
- C3 pad 1: Net-(C3-Pad1) -> Net-(U1-ITH)
- C3 pad 2: Net-(U1-ITH) -> GND
- C4 pad 1: Net-(U1-VFB) -> BPOW
- C4 pad 2: Net-(U1-ITH) -> GND
- C5 pad 1: Net-(U1-SENSE+) -> GND
- C5 pad 2: Net-(D1-K) -> 3V3
- C6 pad 1: Net-(D1-A) -> GND
- C6 pad 2: GND -> 5.5V
- C7 pad 1: Net-(U1-EXTVCC) -> 5.5V
- C8 pad 1: Net-(U2-VOUT) -> 3V3
- D1 pad 2: Net-(D1-A) -> GND
- D2 pad A: GND -> Net-(D2-PadA)
- J1 pad A1: unconnected-(J1-~{PRSNT1}-PadA1) -> TD-IN
- J1 pad A10: Net-(J1-+3.3V-PadA10) -> A429-
- J1 pad A11: unconnected-(J1-~{PERST}-PadA11) -> A429+
- J1 pad A12: Net-(J1-GND-PadA12) -> SOUT1
- J1 pad A13: unconnected-(J1-REFCLK+-PadA13) -> SOUT2
- J1 pad A14: unconnected-(J1-REFCLK--PadA14) -> SIN1
- J1 pad A15: Net-(J1-GND-PadA12) -> SIN2
- J1 pad A16: unconnected-(J1-PERp0-PadA16) -> GND
- J1 pad A17: unconnected-(J1-PERn0-PadA17) -> BPOW
- J1 pad A18: Net-(J1-GND-PadA12) -> GND
- J1 pad A19: unconnected-(J1-RSVD-PadA19) -> DSI1
- J1 pad A2: Net-(J1-+12V-PadA2) -> TD+IN
- J1 pad A20: Net-(J1-GND-PadA12) -> DSI2
- J1 pad A21: unconnected-(J1-PERp1-PadA21) -> DSI3
- J1 pad A22: unconnected-(J1-PERn1-PadA22) -> DSI4
- J1 pad A23: Net-(J1-GND-PadA12) -> DSI5
- J1 pad A24: Net-(J1-GND-PadA12) -> DSI6
- J1 pad A25: unconnected-(J1-PERp2-PadA25) -> GND
- J1 pad A26: unconnected-(J1-PERn2-PadA26) -> GND
- J1 pad A27: Net-(J1-GND-PadA12) -> DOFB1
- J1 pad A28: Net-(J1-GND-PadA12) -> DOFB2
- J1 pad A29: unconnected-(J1-PERp3-PadA29) -> DOFB3
- J1 pad A3: Net-(J1-+12V-PadA2) -> RTD-IN
- J1 pad A30: unconnected-(J1-PERn3-PadA30) -> DOFB4
- J1 pad A31: Net-(J1-GND-PadA12) -> DOFB5
- J1 pad A32: unconnected-(J1-RSVD-PadA32) -> DOFB6
- J1 pad A33: unconnected-(J1-RSVD-PadA33) -> GND
- J1 pad A34: Net-(J1-GND-PadA12) -> Net-(J1-PadA34)
- J1 pad A35: unconnected-(J1-PERp4-PadA35) -> Net-(J1-PadA35)
- J1 pad A36: unconnected-(J1-PERn4-PadA36) -> Net-(J1-PadA36)
- J1 pad A37: Net-(J1-GND-PadA12) -> unconnected-(J1-PadA37)
- J1 pad A38: Net-(J1-GND-PadA12) -> unconnected-(J1-PadA38)
- J1 pad A4: Net-(J1-GND-PadA12) -> RTD+IN
- J1 pad A41: Net-(J1-GND-PadA12) -> unconnected-(J1-PadA41)
- J1 pad A42: Net-(J1-GND-PadA12) -> unconnected-(J1-PadA42)
- J1 pad A45: Net-(J1-GND-PadA12) -> unconnected-(J1-PadA45)
- J1 pad A46: Net-(J1-GND-PadA12) -> unconnected-(J1-PadA46)
- J1 pad A49: Net-(J1-GND-PadA12) -> unconnected-(J1-PadA49)
- J1 pad A5: unconnected-(J1-JTAG2-PadA5) -> DAC_OUT
- J1 pad A6: unconnected-(J1-JTAG3-PadA6) -> GND
- J1 pad A7: unconnected-(J1-JTAG4-PadA7) -> CANHI
- J1 pad A8: unconnected-(J1-JTAG5-PadA8) -> CANLO
- J1 pad A9: Net-(J1-+3.3V-PadA10) -> GND
- J1 pad B1: Net-(J1-+12V-PadA2) -> TD-IN
- J1 pad B10: unconnected-(J1-3.3Vaux-PadB10) -> A429-
- J1 pad B11: unconnected-(J1-~{WAKE}-PadB11) -> A429+
- J1 pad B12: unconnected-(J1-RSVD-PadB12) -> SOUT1
- J1 pad B13: Net-(J1-GND-PadA12) -> SOUT2
- J1 pad B14: unconnected-(J1-PETp0-PadB14) -> SIN1
- J1 pad B15: unconnected-(J1-PETn0-PadB15) -> SIN2
- J1 pad B16: Net-(J1-GND-PadA12) -> GND
- J1 pad B17: unconnected-(J1-~{PRSNT2}-PadB17) -> BPOW
- J1 pad B18: Net-(J1-GND-PadA12) -> GND
- J1 pad B19: unconnected-(J1-PETp1-PadB19) -> DSI1
- J1 pad B2: Net-(J1-+12V-PadA2) -> TD+IN
- J1 pad B20: unconnected-(J1-PETn1-PadB20) -> DSI2
- J1 pad B21: Net-(J1-GND-PadA12) -> DSI3
- J1 pad B22: Net-(J1-GND-PadA12) -> DSI4
- J1 pad B23: unconnected-(J1-PETp2-PadB23) -> DSI5
- J1 pad B24: unconnected-(J1-PETn2-PadB24) -> DSI6
- J1 pad B25: Net-(J1-GND-PadA12) -> GND
- J1 pad B26: Net-(J1-GND-PadA12) -> GND
- J1 pad B27: unconnected-(J1-PETp3-PadB27) -> DOFB1
- J1 pad B28: unconnected-(J1-PETn3-PadB28) -> DOFB2
- J1 pad B29: Net-(J1-GND-PadA12) -> DOFB3
- J1 pad B3: Net-(J1-+12V-PadA2) -> RTD-IN
- J1 pad B30: unconnected-(J1-RSVD-PadB30) -> DOFB4
- J1 pad B31: unconnected-(J1-~{PRSNT2}-PadB31) -> DOFB5
- J1 pad B32: Net-(J1-GND-PadA12) -> DOFB6
- J1 pad B33: unconnected-(J1-PETp4-PadB33) -> GND
- J1 pad B35: Net-(J1-GND-PadA12) -> unconnected-(J1-PadB35)
- J1 pad B36: Net-(J1-GND-PadA12) -> unconnected-(J1-PadB36)
- J1 pad B39: Net-(J1-GND-PadA12) -> unconnected-(J1-PadB39)
- J1 pad B4: Net-(J1-GND-PadA12) -> RTD+IN
- J1 pad B40: Net-(J1-GND-PadA12) -> unconnected-(J1-PadB40)
- J1 pad B43: Net-(J1-GND-PadA12) -> unconnected-(J1-PadB43)
- J1 pad B44: Net-(J1-GND-PadA12) -> unconnected-(J1-PadB44)
- J1 pad B47: Net-(J1-GND-PadA12) -> unconnected-(J1-PadB47)
- J1 pad B49: Net-(J1-GND-PadA12) -> unconnected-(J1-PadB49)
- J1 pad B5: unconnected-(J1-SMCLK-PadB5) -> DAC_OUT
- J1 pad B6: unconnected-(J1-SMDAT-PadB6) -> GND
- J1 pad B7: Net-(J1-GND-PadA12) -> CANHI
- J1 pad B8: Net-(J1-+3.3V-PadA10) -> CANLO
- J1 pad B9: unconnected-(J1-JTAG1-PadB9) -> GND
- L1 pad 2: Net-(U1-EXTVCC) -> Net-(D1-K)
- R1 pad 1: Net-(C2-Pad1) -> Net-(U1-FREQ)
- R1 pad 2: GND -> Net-(R1-Pad2)
- R10 pad 1: GND -> Net-(U10-PG)
- R10 pad 2: Net-(U2-VOUT) -> 5.5V
- R11 pad 1: Net-(U2-VOUT) -> Net-(R11-Pad1)
- R11 pad 2: Net-(U2-PG) -> 5.5V
- R12 pad 1: Net-(D3-K) -> Net-(D2-PadA)
- R12 pad 2: Net-(D4-K) -> Net-(R12-Pad2)
- R13 pad 2: Net-(R13-Pad2) -> DSI1
- R14 pad 1: Net-(D5-A) -> Net-(R14-Pad1)
- R14 pad 2: Net-(D5-K) -> DI2
- R15 pad 2: Net-(R15-Pad2) -> DSI2
- R16 pad 1: Net-(D7-A) -> Net-(R16-Pad1)
- R16 pad 2: Net-(D7-K) -> DI3
- R17 pad 2: Net-(R17-Pad2) -> DSI3
- R18 pad 1: Net-(D10-K) -> Net-(R18-Pad1)
- R18 pad 2: Net-(D9-K) -> DI4
- R19 pad 2: Net-(R19-Pad2) -> DSI4
- R2 pad 1: Net-(C3-Pad1) -> BPOW
- R2 pad 2: Net-(U1-VFB) -> Net-(U1-SENSE+)
- R20 pad 1: Net-(D11-A) -> Net-(R20-Pad1)
- R20 pad 2: Net-(D11-K) -> DI5
- R21 pad 2: Net-(R21-Pad2) -> DSI5
- R22 pad 1: Net-(D13-A) -> Net-(R22-Pad1)
- R22 pad 2: Net-(D13-K) -> DI6
- R23 pad 2: Net-(R23-Pad2) -> DSI6
- R3 pad 1: Net-(U1-PGOOD) -> Net-(R3-Pad1)
- R3 pad 2: Net-(D1-A) -> BPOW
- R4 pad 1: Net-(MOSFET1-G) -> Net-(R4-Pad1)
- R4 pad 2: Net-(U1-ION) -> Net-(U1-PGUV)
- R5 pad 1: Net-(MOSFET1-G) -> GND
- R5 pad 2: Net-(U1-NDRV) -> 28V_REF
- R6 pad 1: Net-(U1-VFB) -> Net-(R6-Pad1)
- R6 pad 2: Net-(U1-EXTVCC) -> 3V3
- R7 pad 2: Net-(U1-VFB) -> Net-(U9-SENSE/ADJ)
- R8 pad 1: Net-(U2-SENSE/ADJ) -> Net-(U9-PG)
- R8 pad 2: Net-(U2-VOUT) -> 3V3
- R9 pad 1: GND -> Net-(R66-Pad2)
- R9 pad 2: Net-(U2-SENSE/ADJ) -> 3V3
- U1 pad 1: Net-(U1-ION) -> Net-(U1-GATE)
- U1 pad 10: Net-(U1-PL/LPF) -> Net-(U1-TRACK/SS)
- U1 pad 11: Net-(U1-SS/TRACK) -> GND
- U1 pad 12: GND -> unconnected-(U1-PGOOD-Pad12)
- U1 pad 13: Net-(D1-A) -> Net-(U1-FREQ)
- U1 pad 14: Net-(D1-A) -> GND
- U1 pad 15: Net-(U1-NDRV) -> GND
- U1 pad 16: Net-(U1-EXTVCC) -> unconnected-(U1-DRVUV/EXTG-Pad16)
- U1 pad 18: Net-(D1-A) -> Net-(U1-CAP)
- U1 pad 20: GND -> 28V_REF
- U1 pad 3: unconnected-(U1-NC_3-Pad3) -> 28V_REF
- U1 pad 5: Net-(D1-A) -> Net-(U1-SENSE+)
- U1 pad 6: Net-(U1-PGOOD) -> BPOW
- U1 pad 7: GND -> Net-(U1-ITH)
- U1 pad 8: Net-(U1-ITH) -> Net-(U1-PGUV)
- U1 pad 9: Net-(U1-VFB) -> Net-(U1-PGUV)
- U2 pad 1: Net-(U2-VOUT) -> unconnected-(U2-Pad1)
- U2 pad 2: Net-(U2-SENSE/ADJ) -> unconnected-(U2-Pad2)
- U2 pad 3: GND -> Net-(D1-K)
- U2 pad 4: unconnected-(U2-NC-Pad4) -> Net-(U1-GATE)
- U2 pad 5: Net-(U2-EN/UVLO) -> unconnected-(U2-Pad5)
- U2 pad 6: GND -> unconnected-(U2-Pad6)
- U2 pad 7: Net-(U2-PG) -> unconnected-(U2-Pad7)
- U2 pad 8: Net-(U2-EN/UVLO) -> 28V_REF
- U3 pad 1: Net-(D3-K) -> Net-(D2-PadA)
- U3 pad 3: Net-(R13-Pad2) -> DSI1
- U3 pad 4: Net-(U2-VOUT) -> 3V3
- U4 pad 1: Net-(D5-A) -> Net-(D15-PadC)
- U4 pad 3: Net-(R15-Pad2) -> DSI2
- U4 pad 4: unconnected-(U4-Pad4) -> 3V3
- U5 pad 1: Net-(D7-A) -> Net-(D4-PadA)
- U5 pad 3: Net-(R17-Pad2) -> DSI3
- U5 pad 4: unconnected-(U5-Pad4) -> 3V3
- U6 pad 1: Net-(D10-K) -> Net-(D7-PadA)
- U6 pad 3: Net-(R19-Pad2) -> DSI4
- U6 pad 4: unconnected-(U6-Pad4) -> 3V3
- U7 pad 1: Net-(D11-A) -> Net-(D10-PadC)
- U7 pad 3: Net-(R21-Pad2) -> DSI5
- U7 pad 4: unconnected-(U7-Pad4) -> 3V3
- U8 pad 1: Net-(D13-A) -> Net-(D11-PadA)
- U8 pad 3: Net-(R23-Pad2) -> DSI6
- U8 pad 4: unconnected-(U8-Pad4) -> 3V3
Routing:
- net GND: track 6.86 -> 408.9 mm, vias 3 -> 211
- net TD+IN: track 0.00 -> 307.4 mm, vias 0 -> 1
- net CANLO: track 0.00 -> 295.7 mm, vias 0 -> 2
- net RTD+IN: track 0.00 -> 295.7 mm, vias 0 -> 1
- net A429-: track 0.00 -> 288.8 mm, vias 0 -> 2
- net SOUT1: track 0.00 -> 285.3 mm, vias 0 -> 4
- net TD-IN: track 0.00 -> 200.1 mm, vias 0 -> 1
- net A429+: track 0.00 -> 198.0 mm, vias 0 -> 1
- net SOUT2: track 0.00 -> 193.2 mm, vias 0 -> 2
- net CANHI: track 0.00 -> 191.3 mm
- net SIN2: track 0.00 -> 191.3 mm, vias 0 -> 1
- net RTD-IN: track 0.00 -> 189.4 mm, vias 0 -> 1
- net DAC_OUT: track 0.00 -> 185.2 mm, vias 0 -> 1
- net SIN1: track 0.00 -> 166.8 mm, vias 0 -> 4
- net DOFB1: track 0.00 -> 145.9 mm, vias 0 -> 1
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- added copper zone on In2.Cu, net 28V_REF
- added copper zone on In2.Cu, net 3V3
- added copper zone on In2.Cu, net 5.5V
- added copper zone on In2.Cu, net BPOW
- added copper zone on In1.Cu, net GND
- removed copper zone on B.Cu, net GND
Other:
- board size 167.6 x 96.5 mm -> 184 x 95 mm
