File: Backplane.kicad_sch (KiCad schematic)
At the start: 58 parts, among them U1 LTC3810IG_PBF, U2 ADP7104ACPZ-3.0-R7, U3 ISP817CXSM, U4 ISP817CXSM, U5 ISP817CXSM, U6 ISP817CXSM, U7 ISP817CXSM, U8 ISP817CXSM

Commit message: Add files via upload
Reworked power supply just needs verification from Tim but PCB is getting set up and much simpler schematic!
Parts:
- removed C6: 1u, Capacitor_THT:CP_Axial_L10.0mm_D4.5mm_P15.00mm_Horizontal, symbol Device:C_Small
- removed C7: 240u, Capacitor_THT:CP_Axial_L10.0mm_D4.5mm_P15.00mm_Horizontal, symbol Device:C_Small
- removed C8: 2.2u, Capacitor_THT:CP_Axial_L10.0mm_D4.5mm_P15.00mm_Horizontal, symbol Device:C_Small
- removed D1: 1N4148, Diode_THT:D_DO-35_SOD27_P7.62mm_Horizontal, symbol Diode:1N4148
- removed D10, D11, D12, D13, D14, D3, D4, D5, D6, D7, D8, D9: MBR745, Package_TO_SOT_THT:TO-220-2_Vertical, symbol Diode:MBR745
- removed D15: 1N4007, Diode_THT:D_DO-41_SOD81_P10.16mm_Horizontal, symbol Diode:1N4007
- removed D2: RB168MM100, SDII Lib:SOD-123FL, symbol RB168MM100:RB168MM100
- removed MOSFET1, MOSFET2, MOSFET3: SI7850DP-T1-E3, SDII Lib:POWERPAK_SO-8_SINGLE_VIS, symbol ADP7104:SI7850DP-T1-E3
- removed R10: 12, Resistor_THT:R_Axial_DIN0204_L3.6mm_D1.6mm_P5.08mm_Horizontal, symbol Device:R_Small_US
- removed R11: 100k, Resistor_THT:R_Axial_DIN0204_L3.6mm_D1.6mm_P5.08mm_Horizontal, symbol Device:R_Small_US
- removed U1: LTC3810IG_PBF, SDII Lib:SSOP-28_G, symbol LTC3810IG_PBF:LTC3810IG_PBF
- removed U2: ADP7104ACPZ-3.0-R7, SDII Lib:CP_8_5_ADI, symbol SI7850DP:ADP7104ACPZ-3.0-R7
- added D1: 1N5818, Diode_THT:D_DO-41_SOD81_P10.16mm_Horizontal, symbol Diode:1N5818
- added D10, D11, D12, D15, D2, D3, D4, D5, D6, D7, D8, D9: 1N4148, Diode_THT:D_DO-35_SOD27_P7.62mm_Horizontal, symbol Diode:1N4148
- added J1, J2, J3, J4, J5: PCIE-098-02-X-D-TH, PCIE-098-02-X-D-TH:SAMTEC_PCIE-098-02-X-D-TH, symbol PCI:PCIE-098-02-X-D-TH
- added U1: LTC3894EFE-PBF, TSSOP20-EP_4P4X6P5_ADI, symbol LTC3894:LTC3894EFE-PBF
- added U2: FDS4435A, SOIC8_751EB_FAS, symbol FDS4435A:FDS4435A
- added U9: ADP7104ACPZ-3.0-R7, CP_8_5_ADI, symbol SI7850DP:ADP7104ACPZ-3.0-R7
- C1: value 560p -> .47u; footprint Capacitor_THT:CP_Axial_L10.0mm_D4.5mm_P15.00mm_Horizontal -> (none)
- C2: value .01u -> 0.1u; footprint Capacitor_THT:CP_Axial_L10.0mm_D4.5mm_P15.00mm_Horizontal -> (none)
- C3: value 220p -> 3.3n; footprint Capacitor_THT:CP_Axial_L10.0mm_D4.5mm_P15.00mm_Horizontal -> (none)
- C4: value 33p -> 330u; footprint Capacitor_THT:CP_Axial_L10.0mm_D4.5mm_P15.00mm_Horizontal -> (none)
- C5: value 0.1u -> 2.2u; footprint Capacitor_THT:CP_Axial_L10.0mm_D4.5mm_P15.00mm_Horizontal -> (none)
- L1: value 7.6u -> 22u; footprint Inductor_SMD:L_Bourns_SRR1260 -> (none)
- R1: value 10k -> 36.5k; footprint Resistor_THT:R_Axial_DIN0204_L3.6mm_D1.6mm_P5.08mm_Horizontal -> (none)
- R12, R13, R14, R15, R16, R17, R18, R19, R20, R21, R22, R23: footprint Resistor_THT:R_Axial_DIN0204_L3.6mm_D1.6mm_P5.08mm_Horizontal -> (none)
- R2: value 90.9k -> 20m; footprint Resistor_THT:R_Axial_DIN0204_L3.6mm_D1.6mm_P5.08mm_Horizontal -> (none)
- R3: value 100k -> 422k; footprint Resistor_THT:R_Axial_DIN0204_L3.6mm_D1.6mm_P5.08mm_Horizontal -> (none)
- R4: value 274k -> 52k; footprint Resistor_THT:R_Axial_DIN0204_L3.6mm_D1.6mm_P5.08mm_Horizontal -> (none)
- R5: value 100k -> 2; footprint Resistor_THT:R_Axial_DIN0204_L3.6mm_D1.6mm_P5.08mm_Horizontal -> (none)
- R6: value 8k -> 17.4k; footprint Resistor_THT:R_Axial_DIN0204_L3.6mm_D1.6mm_P5.08mm_Horizontal -> (none)
- R7: value 1k -> 10k; footprint Resistor_THT:R_Axial_DIN0204_L3.6mm_D1.6mm_P5.08mm_Horizontal -> (none)
- R8: value 8k -> 100k; footprint Resistor_THT:R_Axial_DIN0204_L3.6mm_D1.6mm_P5.08mm_Horizontal -> (none)
- R9: value 1k -> 12; footprint Resistor_THT:R_Axial_DIN0204_L3.6mm_D1.6mm_P5.08mm_Horizontal -> (none)
Connections:
- net GND: now also C2.2, C3.2, C4.2, C5.1, R4.1, R5.1, D1.2 (A), D10.2 (A), D12.2 (A), D15.2 (A), D2.2 (A), D5.2 (A), D8.2 (A), U1.11 (PLLIN/MODE), U1.14 (OVLO), U1.15 (EXTS), U9.3 (GND), U9.6 (GND); no longer C1.1
- net at R16.1, U5.1: now also D4.2 (A), D5.1 (K)
- net at R16.2: now also D4.1 (K)
- net at C2.1: now also U1.10 (TRACK/SS); no longer R1.1
- net at R9.2: now also C5.2, R6.2, R8.2, U3.4, U4.4, U5.4, U6.4, U7.4, U8.4, U9.1 (VOUT); no longer R8.1
- net at R22.1, U8.1: now also D11.2 (A), D12.1 (K)
- net at L1.1: now also R2.2, U1.5 (SENSE+); no longer C5.1
- net at L1.2: now also D1.1 (K), U2.3; no longer R6.2
- net at R20.1, U7.1: now also D10.1 (K), D9.2 (A)
- net at R18.1, U6.1: now also D7.2 (A), D8.1 (K)
- net at R14.2: now also D6.1 (K)
- net at R14.1, U4.1: now also D15.1 (K), D6.2 (A)
- net at R12.1, U3.1: now also D2.1 (K), D3.2 (A)
- net at R3.2: now also C4.1, R2.1, R5.2, U1.6 (SENSE-)
- net at R20.2: now also D9.1 (K)
- net at R12.2: now also D3.1 (K)
- net at R4.2: now also R3.1, U1.8 (PGUV), U1.9 (VFB)
- net at C1.2: now also U1.18 (CAP)
- net at R6.1, R7.2: now also U9.2 (SENSE/ADJ); no longer C4.1, R2.2
- net at R22.2: now also D11.1 (K)
- net at C3.1: now also U1.7 (ITH); no longer R2.1
- net at R18.2: now also D7.1 (K)
- new net: U9.5 (EN/UVLO), U9.8 (VIN)
- new net: R8.1, U9.7 (PG)
- new net: R1.1, U1.13 (FREQ)
- new net: C1.1, U1.20 (VIN), U1.3 (RUN), U2.8
- new net: U1.1 (GATE), U2.4

Commit message: Merged both -1/-2 and backplane
Parts:
- removed D10, D11, D12, D15, D2, D3, D4, D5, D6, D7, D8, D9: 1N4148, Diode_THT:D_DO-35_SOD27_P7.62mm_Horizontal, symbol Diode:1N4148
- removed J1, J2, J3, J4, J5: PCIE-098-02-X-D-TH, PCIE-098-02-X-D-TH:SAMTEC_PCIE-098-02-X-D-TH, symbol PCI:PCIE-098-02-X-D-TH
- removed U9: ADP7104ACPZ-3.0-R7, CP_8_5_ADI, symbol SI7850DP:ADP7104ACPZ-3.0-R7
- added C10, C11, C12, C13, C14, C15, C16, C17, C18, C19, C20, C21, C22, C23, C7, C8, C9: 10u, Capacitor_SMD:C_1206_3216Metric, symbol Device:C_Small
- added C6: 22u, Capacitor_SMD:C_1206_3216Metric, symbol Device:C_Small
- added CR1: SMDJ85A, SDII Lib:SMDJ85A, symbol SMDJ85A:SMDJ85A
- added CR10, CR12, CR14, CR16, CR18, CR19, CR20, CR24, CR25, CR26, CR6, CR8: SMDJ33A, SDII Lib:SMDJ33A, symbol SMDJ33A:SMDJ33A
- added CR27, CR28, CR29, CR30, CR31: SMDJ6.0A, SDII Lib:SMDJ6_0A, symbol SMDJ6.0A:SMDJ6.0A
- added CR32: RF201LAM2STR, SDII Lib:RF201LAM2STR(new_POW_diode), symbol RF201LAM2STR(new_POW_diode):RF201LAM2STR
- added CR33, CR34, CR35, CR36, CR37, CR38, CR39, CR40, CR41, CR42, CR43, CR44: RBR1MM60ATFTR, SDII Lib:RBR1MM60ATFTR(new_VR_diode), symbol RBR1MM60ATFTR(new_VR_diode):RBR1MM60ATFTR
- added D10, D11, D12, D15, D2, D3, D4, D5, D6, D7, D8, D9: 1N4148WS, SDII Lib:1N4148WS, symbol 1N4148:1N4148WS
- added D27, D28, D29, D30, D31, D32, D33, D34, D35, D36: 1N5819HW-7-F, SDII Lib:1N5819, symbol 1N5819:1N5819HW-7-F
- added D37, D38, D39, D40, D41, D42: SMDJ60CA, SDII Lib:SMDJ6_0CA, symbol SMDJ6.0CA:SMDJ60CA
- added H1, H2, H3, H4: MountingHole, MountingHole:MountingHole_3.2mm_M3, symbol Mechanical:MountingHole
- added J1, J2, J3, J4, J5: 10018783-10202TLF, SDII Lib:PCI_Express_Card, symbol PCI_Express:10018783-10202TLF
- added J6: 5019514000, SDII Lib:BP_Connector, symbol BP_Connector:5019514000
- added R10: 100k, Resistor_SMD:R_0805_2012Metric, symbol Device:R_Small_US
- added R100, R27, R29, R31, R33, R35, R37, R86, R87, R88, R89, R90, R92, R94, R95, R99: 1k, Resistor_SMD:R_0805_2012Metric, symbol Device:R_Small_US
- added R11: 10, Resistor_SMD:R_0805_2012Metric, symbol Device:R_Small_US
- added R24: 15k, Resistor_SMD:R_0805_2012Metric, symbol Device:R_Small_US
- added R25: 4.7k, Resistor_SMD:R_0805_2012Metric, symbol Device:R_Small_US
- added R26, R28, R30, R32, R34, R36, R68, R83: 3k, Resistor_SMD:R_0805_2012Metric, symbol Device:R_Small_US
- added R38, R39, R40, R41, R42, R43, R44, R45, R46, R47, R48, R49: 1K, Resistor_SMD:R_0805_2012Metric, symbol Device:R_Small_US
- added R50, R51, R52, R53, R54: 100K, Resistor_SMD:R_0805_2012Metric, symbol Device:R_Small_US
- added R55, R56, R57, R58, R59, R60: 10K, Resistor_SMD:R_0805_2012Metric, symbol Device:R_Small_US
- added R61, R63: 2.2k, Resistor_SMD:R_0805_2012Metric, symbol Device:R_Small_US
- added R62, R64, R65: 200, Resistor_SMD:R_0402_1005Metric, symbol Device:R_Small_US
- added R66, R67: 2, Resistor_SMD:R_0603_1608Metric, symbol Device:R_Small_US
- added R69, R70, R71, R72, R73, R74, R75, R76, R77, R78, R79, R84: 2k, Resistor_SMD:R_0805_2012Metric, symbol Device:R_Small_US
- added R80, R82: 22k, Resistor_SMD:R_0805_2012Metric, symbol Device:R_Small_US
- added R81: 200k, Resistor_SMD:R_0805_2012Metric, symbol Device:R_Small_US
- added R85: 1.5k, Resistor_SMD:R_0805_2012Metric, symbol Device:R_Small_US
- added U10, U9: ADP7104ACPZ-R7, SDII Lib:CP_8_5_ADI, symbol ADP7104ACPZ_R7:ADP7104ACPZ-R7
- added U11, U12, U13, U14, U15, U16: ISP817CXSM, SDII Lib:ISP817SM_ISO, symbol ISP817CX:ISP817CXSM
- added U17, U18, U19, U20, U21: OP191GSZ-REEL7, SDII Lib:OP191, symbol OP191:OP191GSZ-REEL7
- C1: footprint (none) -> Capacitor_SMD:C_0805_2012Metric
- C2, C3: footprint (none) -> Capacitor_SMD:C_0603_1608Metric
- C4: value 330u -> 33u; footprint (none) -> Capacitor_SMD:C_1206_3216Metric
- C5: value 2.2u -> 22u; footprint (none) -> Capacitor_SMD:C_1206_3216Metric
- L1: footprint (none) -> SDII Lib:IND_1210-WE-PD_WRE
- R1: value 36.5k -> 30k; footprint (none) -> Resistor_SMD:R_0805_2012Metric
- R12: value 5k -> 2k; footprint (none) -> Resistor_SMD:R_0805_2012Metric
- R13, R15, R17, R19, R21, R23, R7, R8: footprint (none) -> Resistor_SMD:R_0805_2012Metric
- R14, R16, R18, R20, R22: value 5k -> 3k; footprint (none) -> Resistor_SMD:R_0805_2012Metric
- R2: footprint (none) -> Resistor_SMD:R_1206_3216Metric
- R3: value 422k -> 200k; footprint (none) -> Resistor_SMD:R_0805_2012Metric
- R4: value 52k -> 30k; footprint (none) -> Resistor_SMD:R_0805_2012Metric
- R5: value 2 -> 10K; footprint (none) -> Resistor_SMD:R_0805_2012Metric
- R6: value 17.4k -> 15k; footprint (none) -> Resistor_SMD:R_0805_2012Metric
- R9: value 12 -> 10; footprint (none) -> Resistor_SMD:R_0805_2012Metric
- U1: footprint TSSOP20-EP_4P4X6P5_ADI -> SDII Lib:TSSOP20-EP_4P4X6P5_ADI
- U2: footprint SOIC8_751EB_FAS -> SDII Lib:SOIC8_751EB_FAS
Connections:
- net GND: now also C10.2, C11.2, C12.2, C13.2, C14.2, C15.2, C16.2, C17.2, C18.2, C19.2, C20.2, C21.2, C22.2, C23.2, C6.1, C7.2, C8.2, C9.2, CR1.2, CR10.2, CR12.2, CR14.2, CR16.2, CR18.2, CR19.2, CR20.2, CR24.2, CR25.2, CR26.2, CR27.2, CR28.2, CR29.2, CR30.2, CR31.2, CR32.2, CR33.2, CR34.2, CR35.2, CR36.2, CR37.2, CR38.2, CR39.2, CR40.2, CR41.2, CR42.2, CR43.2, CR44.2, CR6.2, CR8.2, D10.A, D12.A, D15.A, D27.A, D29.A, D3.A, D31.A, D33.A, D35.A, D37.1, D38.1, D39.1, D40.1, D41.1, D42.1, D5.A, D8.A, J1.A16, J1.A18, J1.A25, J1.A26, J1.A33, J1.A6, J1.A9, J1.B16, J1.B18, J1.B25, J1.B26, J1.B33, J1.B6, J1.B9, J2.A16, J2.A18, J2.A25, J2.A26, J2.A33, J2.A6, J2.A9, J2.B16, J2.B18, J2.B25, J2.B26, J2.B33, J2.B6, J2.B9, J3.A16, J3.A18, J3.A25, J3.A26, J3.A33, J3.A6, J3.A9, J3.B16, J3.B18, J3.B25, J3.B26, J3.B33, J3.B6, J3.B9, J4.A16, J4.A18, J4.A25, J4.A26, J4.A33, J4.A6, J4.A9, J4.B16, J4.B18, J4.B25, J4.B26, J4.B33, J4.B6, J4.B9, J5.A16, J5.A18, J5.A25, J5.A26, J5.A33, J5.A6, J5.A9, J6.16, J6.18, J6.25, J6.26, J6.33, J6.6, J6.9, R100.1, R27.1, R29.1, R31.1, R33.1, R35.1, R37.1, R38.1, R39.1, R40.1, R41.1, R42.1, R43.1, R44.1, R45.1, R46.1, R47.1, R48.1, R49.1, R50.1, R51.1, R52.1, R53.1, R54.1, R55.1, R56.1, R57.1, R58.1, R59.1, R60.1, R65.1, R66.1, R67.1, R80.1, R85.2, R86.1, R87.1, R88.1, R89.1, R90.1, R92.1, R94.1, R95.1, R99.1, U10.3 (GND), U10.6 (GND), U10.9 (EPAD), U11.2, U12.2, U13.2, U14.2, U15.2, U16.2, U17.4 (-V), U18.4 (-V), U19.4 (-V), U20.4 (-V), U21.4 (-V), U9.3 (GND), U9.6 (GND), U9.9 (EPAD); no longer R1.2, R4.1, R9.1
- net at U5.1: now also D4.A, D5.C, R70.1; no longer R16.1
- net DI3: now reaches R16.2
- net DI3: now also CR14.1, CR35.1, J6.21, R43.2
- net at U8.1: now also D11.A, D12.C, R73.1; no longer R22.1
- net 3V3: now reaches C5.2, R6.2, R8.2, R9.2, U3.4, U4.4, U5.4, U6.4, U7.4, U8.4
- net 3V3: now also C10.1, C11.1, C12.1, C13.1, C8.1, C9.1, U9.1 (VOUT)
- net at R7.2: now also R62.1, U9.2 (SENSE/ADJ); no longer R6.1
- net at R8.1: now also U9.7 (PG)
- net DSI6: now reaches R23.2, U8.3
- net DSI6: now also J1.A24, J1.B24, J2.A24, J2.B24, J3.A24, J3.B24, J4.A24, J4.B24, J5.A24
- net DI4: now reaches R18.2
- net DI4: now also CR36.1, CR8.1, J6.22, R40.2
- net at U6.1: now also D7.A, D8.C, R71.1; no longer R18.1
- net at R4.2, U1.8 (PGUV), U1.9 (VFB): now also R82.1; no longer R3.1
- net DI6: now reaches R22.2
- net DI6: now also CR16.1, CR38.1, J6.24, R44.2
- net at R12.1, U3.1: now also D2.A, D3.C
- net DSI1: now reaches R13.2, U3.3
- net DSI1: now also J1.A19, J1.B19, J2.A19, J2.B19, J3.A19, J3.B19, J4.A19, J4.B19, J5.A19
- net at U7.1: now also D10.C, D9.A, R72.1; no longer R20.1
- net at R12.2: now also R68.1
- net DSI3: now reaches R17.2, U5.3
- net DSI3: now also J1.A21, J1.B21, J2.A21, J2.B21, J3.A21, J3.B21, J4.A21, J4.B21, J5.A21
- net at U4.1: now also D15.C, D6.A, R69.1; no longer R14.1
- net DI2: now reaches R14.2
- net DI2: now also CR10.1, CR34.1, J6.20, R41.2
- net BPOW: now reaches C4.1, R2.1, R3.2, U1.6 (SENSE-)
- net BPOW: now also J1.A17, J1.B17, J2.A17, J2.B17, J3.A17, J3.B17, J4.A17, J4.B17, J5.A17, U10.5 (EN/UVLO), U10.8 (VIN), U9.5 (EN/UVLO), U9.8 (VIN); no longer R5.2
- net DSI4: now reaches R19.2, U6.3
- net DSI4: now also J1.A22, J1.B22, J2.A22, J2.B22, J3.A22, J3.B22, J4.A22, J4.B22, J5.A22
- net DI5: now reaches R20.2
- net DI5: now also CR12.1, CR37.1, J6.23, R42.2
- net DSI5: now reaches R21.2, U7.3
- net DSI5: now also J1.A23, J1.B23, J2.A23, J2.B23, J3.A23, J3.B23, J4.A23, J4.B23, J5.A23
- net DSI2: now reaches R15.2, U4.3
- net DSI2: now also J1.A20, J1.B20, J2.A20, J2.B20, J3.A20, J3.B20, J4.A20, J4.B20, J5.A20
- net 28V_REF: now reaches C1.1, U1.20 (VIN), U1.3 (RUN), U2.8
- net 28V_REF: now also R5.2, C14.1, C15.1, C16.1, C17.1, C18.1, C19.1, CR1.1, CR32.1, D11.C, D2.C, D4.C, D6.C, D7.C, D9.C, J6.17, U11.4, U12.4, U13.4, U14.4, U15.4, U16.4
- new net: R77.1, U13.1
- new net: CR27.1, J6.1, R50.2, U17.3 (+INA)
- new net: D31.C, D32.A
- new net: D27.C, D28.A
- new net: J1.A36, R88.2
- new net: R79.1, U11.1
- new net: J5.A35, R99.2
- new net: J5.A36, R100.2
- new net: R66.2, R9.1
- new net: J2.A34, R89.2
- new net: D35.C, D36.A
- new net: CR31.1, J6.5, R54.2, U21.3 (+INA)
- new net: R14.1, R69.2
- new net: R75.1, U15.1
- new net: R76.1, U14.1
- new net: R32.1, R76.2
- new net: R74.1, U16.1
- new net: R61.1, R62.2
- new net: R4.1, R80.2
- new net: CR29.1, J6.3, R52.2, U19.3 (+INA)
- new net: CR28.1, J6.2, R51.2, U18.3 (+INA)
- new net: CR30.1, J6.4, R53.2, U20.3 (+INA)
- new net: R11.1, R67.2
- new net: R81.1, R82.2
- new net: R6.1, R61.2
- new net: J3.A36, R94.2
- new net: R28.1, R78.2
- new net: R30.1, R77.2
- new net: R22.1, R73.2
- new net: J2.A35, R90.2
- new net: R25.2, R64.1, U10.2 (SENSE/ADJ)
- new net: R63.1, R64.2
- new net: R1.2, R83.1
- new net: R16.1, R70.2
- new net: J3.A34, R92.2
- new net: R34.1, R75.2
- new net: R24.1, R63.2
- new net: R20.1, R72.2
- new net: R25.1, R65.2
- new net: D29.C, D30.A
- new net: J1.A34, R86.2
- new net: D33.C, D34.A
- new net: J1.A35, R87.2
- new net: R3.1, R81.2
- new net: R78.1, U12.1
- new net: R10.1, U10.7 (PG)
- new net: R83.2, R84.1
- new net: R26.1, R79.2
- new net: R18.1, R71.2
- new net: R84.2, R85.1
- new net: R36.1, R74.2
- new net: J4.A34, R95.2
- new net 5.5V: C20.1, C21.1, C22.1, C23.1, C6.2, C7.1, D28.C, D30.C, D32.C, D34.C, D36.C, R10.2, R11.2, R24.2, U10.1 (VOUT), U17.7 (+V), U18.7 (+V), U19.7 (+V), U20.7 (+V), U21.7 (+V)
- new net A429+: D38.2, J1.A11, J1.B11, J2.A11, J2.B11, J3.A11, J3.B11, J4.A11, J4.B11, J5.A11, J6.11, R56.2
- new net A429-: D37.2, J1.A10, J1.B10, J2.A10, J2.B10, J3.A10, J3.B10, J4.A10, J4.B10, J5.A10, J6.10, R55.2
- new net CANHI: J1.A7, J1.B7, J2.A7, J2.B7, J3.A7, J3.B7, J4.A7, J4.B7, J5.A7
- new net CANLO: J1.A8, J1.B8, J2.A8, J2.B8, J3.A8, J3.B8, J4.A8, J4.B8, J5.A8
- new net DAC_OUT: J1.A5, J1.B5, J2.A5, J2.B5, J3.A5, J3.B5, J4.A5, J4.B5, J5.A5, U21.2 (-INA), U21.6 (OUTA)
- new net DI1: CR33.1, CR6.1, J6.19, R39.2, R68.2
- new net DO1: CR18.1, CR39.1, J6.27, R27.2, R38.2, U11.3
- new net DO2: CR19.1, CR40.1, J6.28, R29.2, R45.2, U12.3
- new net DO3: CR20.1, CR41.1, J6.29, R31.2, R46.2, U13.3
- new net DO4: CR24.1, CR42.1, J6.30, R33.2, R47.2, U14.3
- new net DO5: CR25.1, CR43.1, J6.31, R35.2, R48.2, U15.3
- new net DO6: CR26.1, CR44.1, J6.32, R37.2, R49.2, U16.3
- new net DOFB1: J1.A27, J1.B27, J2.A27, J2.B27, J3.A27, J3.B27, J4.A27, J4.B27, J5.A27, R26.2
- new net DOFB2: J1.A28, J1.B28, J2.A28, J2.B28, J3.A28, J3.B28, J4.A28, J4.B28, J5.A28, R28.2
- new net DOFB3: J1.A29, J1.B29, J2.A29, J2.B29, J3.A29, J3.B29, J4.A29, J4.B29, J5.A29, R30.2
- new net DOFB4: J1.A30, J1.B30, J2.A30, J2.B30, J3.A30, J3.B30, J4.A30, J4.B30, J5.A30, R32.2
- new net DOFB5: J1.A31, J1.B31, J2.A31, J2.B31, J3.A31, J3.B31, J4.A31, J4.B31, J5.A31, R34.2
- new net DOFB6: J1.A32, J1.B32, J2.A32, J2.B32, J3.A32, J3.B32, J4.A32, J4.B32, J5.A32, R36.2
- new net RTD+IN: J1.A4, J1.B4, J2.A4, J2.B4, J3.A4, J3.B4, J4.A4, J4.B4, J5.A4, U20.2 (-INA), U20.6 (OUTA)
- new net RTD-IN: J1.A3, J1.B3, J2.A3, J2.B3, J3.A3, J3.B3, J4.A3, J4.B3, J5.A3, U19.2 (-INA), U19.6 (OUTA)
- new net SIN1: D41.2, J1.A14, J1.B14, J2.A14, J2.B14, J3.A14, J3.B14, J4.A14, J4.B14, J5.A14, J6.14, R59.2
- new net SIN2: D42.2, J1.A15, J1.B15, J2.A15, J2.B15, J3.A15, J3.B15, J4.A15, J4.B15, J5.A15, J6.15, R60.2
- new net SOUT1: D39.2, J1.A12, J1.B12, J2.A12, J2.B12, J3.A12, J3.B12, J4.A12, J4.B12, J5.A12, J6.12, R57.2
- new net SOUT2: D40.2, J1.A13, J1.B13, J2.A13, J2.B13, J3.A13, J3.B13, J4.A13, J4.B13, J5.A13, J6.13, R58.2
- new net TD+IN: J1.A2, J1.B2, J2.A2, J2.B2, J3.A2, J3.B2, J4.A2, J4.B2, J5.A2, U18.2 (-INA), U18.6 (OUTA)
- new net TD-IN: J1.A1, J1.B1, J2.A1, J2.B1, J3.A1, J3.B1, J4.A1, J4.B1, J5.A1, U17.2 (-INA), U17.6 (OUTA)
Other:
- moved on the sheet: C1, C2, C3, C4, C5, D1, L1, R1, R12, R13, R15, R17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
