File: PCB_Test_Jig/PCB_Test_Jig.kicad_sch (KiCad schematic)
At the start: 3 parts, among them J1 10018783-10202TLF

Commit message: Updated the test jig
Parts:
- added D1, D2, D3, D4, D5, D6: LED, LED_SMD:LED_0805_2012Metric, symbol Device:LED
- added J2, J3, J4, J5, J6, J7, J8: Conn_01x02_Pin, SDII LIB:pin header, symbol Connector:Conn_01x02_Pin
- added R1, R2, R3, R4, R5, R6: 1.5k, Resistor_SMD:R_0805_2012Metric, symbol Device:R
- added R7, R8, R9: 1k, Resistor_SMD:R_0805_2012Metric, symbol Device:R
- added S2, S3, S4: TS09-63-25-WT-260-SMT-TR, SDII LIB:SW_TS09-63-25-WT-260-SMT-TR, symbol Single Button:TS09-63-25-WT-260-SMT-TR
- renumbered S2 to S1, S1 to S5
Connections:
- net TD-: now reaches J1.A1
- net TD-: now also J1.B1, J6.2 (Pin_2)
- net A429_IN+: now reaches J1.A10
- net A429_IN+: now also J1.B10, J3.2 (Pin_2)
- net A429_IN-: now reaches J1.A11
- net A429_IN-: now also J1.B11, J3.1 (Pin_1)
- net A429_OUT+: now reaches J1.A12
- net A429_OUT+: now also J1.B12, J2.2 (Pin_2)
- net A429_OUT-: now reaches J1.A13
- net A429_OUT-: now also J1.B13, J2.1 (Pin_1)
- net GND: now reaches J1.A16
- net GND: now also J1.A18, J1.A25, J1.A26, J1.A33, J1.A6, J1.A9, J1.B16, J1.B18, J1.B25, J1.B26, J1.B33, J1.B6, J1.B9, S1.1A, S1.2A, S1.3A, S5.1A, S5.2A, S5.3A, D1.1 (K), D2.1 (K), D3.1 (K), D4.1 (K), D5.1 (K), D6.1 (K), J7.1 (Pin_1), J8.1 (Pin_1), S2.1, S3.1, S4.1
- net VCC: now reaches J1.A17
- net VCC: now also J1.B17, J8.2 (Pin_2)
- net DSI1: now reaches J1.A19
- net DSI1: now also J1.B19, S1.1B
- net TD+: now reaches J1.A2
- net TD+: now also J1.B2, J6.1 (Pin_1)
- net DSI2: now reaches J1.A20
- net DSI2: now also J1.B20, S1.2B
- net DSI3: now reaches J1.A21
- net DSI3: now also J1.B21, S1.3B
- net DIS4: now reaches J1.A22
- net DIS4: now also J1.B22, S2.2
- net DSI5: now reaches J1.A23
- net DSI5: now also J1.B23, S3.2
- net DSI6: now reaches J1.A24
- net DSI6: now also J1.B24, S4.2
- net DOFB1: now reaches J1.A27
- net DOFB1: now also J1.B27, R1.1
- net DOFB2: now reaches J1.A28
- net DOFB2: now also J1.B28, R2.1
- net DOFB3: now reaches J1.A29
- net DOFB3: now also J1.B29, R3.1
- net RTD-: now reaches J1.A3
- net RTD-: now also J1.B3, J5.2 (Pin_2)
- net DOFB4: now reaches J1.A30
- net DOFB4: now also J1.B30, R4.1
- net DOFB5: now reaches J1.A31
- net DOFB5: now also J1.B31, R5.1
- net DOFB6: now reaches J1.A32
- net DOFB6: now also J1.B32, R6.1
- net HW_ID_1: now reaches J1.A34
- net HW_ID_1: now also J1.B34, R7.1
- net HW_ID_2: now reaches J1.A35
- net HW_ID_2: now also J1.B35, R8.1
- net HW_ID_3: now reaches J1.A36
- net HW_ID_3: now also J1.B36, R9.1
- net RTD+: now reaches J1.A4
- net RTD+: now also J1.B4, J5.1 (Pin_1)
- net DAC_OUT: now reaches J1.A5
- net DAC_OUT: now also J1.B5, J7.2 (Pin_2)
- net A825_CAN_HI: now reaches J1.A7
- net A825_CAN_HI: now also J1.B7, J4.2 (Pin_2)
- net A825_CAN_LO: now reaches J1.A8
- net A825_CAN_LO: now also J1.B8, J4.1 (Pin_1)
- net at S5.1B: now also R7.2
- net at S5.2B: now also R8.2
- net at S5.3B: now also R9.2
- new net: D3.2 (A), R3.2
- new net: D6.2 (A), R6.2
- new net: D1.2 (A), R1.2
- new net: D5.2 (A), R5.2
- new net: D2.2 (A), R2.2
- new net: D4.2 (A), R4.2
- no-connect marks 0 -> 30
Other:
- moved on the sheet: J1, S1, S5
