File: Backplane PCB/Backplane.kicad_pcb (KiCad board)
At the start: 4 copper layers, 184 x 95 mm, 213 parts, among them J1 10018783-10202TLF, J2 10018783-10202TLF, J3 10018783-10202TLF, J4 10018783-10202TLF, J5 10018783-10202TLF, J6 5019514000, U1 LTC3894EFE-PBF, U10 ADP7104ACPZ-R7, U11 ISP817CXSM, U12 ISP817CXSM, U13 ISP817CXSM, U14 ISP817CXSM, U15 ISP817CXSM, U16 ISP817CXSM, U17 OP191GSZ-REEL7, U18 OP191GSZ-REEL7, U19 OP191GSZ-REEL7, U2 FDS4435A, U20 OP191GSZ-REEL7, U21 OP191GSZ-REEL7, U3 ISP817CXSM, U4 ISP817CXSM, U5 ISP817CXSM, U6 ISP817CXSM, U7 ISP817CXSM, U8 ISP817CXSM, U9 ADP7104ACPZ-R7

Commit message: Adjusted pins connections names
Connections:
- D39 pad 2: A429_OUT- -> A429_OUT+
- J1 pad A12: A429_OUT- -> A429_OUT+
- J1 pad B12: A429_OUT- -> A429_OUT+
- J2 pad A12: A429_OUT- -> A429_OUT+
- J2 pad B12: A429_OUT- -> A429_OUT+
- J3 pad A12: A429_OUT- -> A429_OUT+
- J3 pad B12: A429_OUT- -> A429_OUT+
- J4 pad A12: A429_OUT- -> A429_OUT+
- J4 pad B12: A429_OUT- -> A429_OUT+
- J5 pad A12: A429_OUT- -> A429_OUT+
- J6 pad 12: A429_OUT- -> A429_OUT+
- R57 pad 2: A429_OUT- -> A429_OUT+
Routing:
- net A429_OUT-: track 478.5 -> 193.2 mm, vias 6 -> 2
- net A429_OUT+: track 0.00 -> 285.3 mm, vias 0 -> 4

Commit message: Added logo
Parts:
- added G***: LOGO, SDII Lib:Big_Logo, F.Cu at (301.5, 128.5)
Connections:
- J5 pad B1: unconnected-(J5-PadB1) -> TD-IN
- J5 pad B10: unconnected-(J5-PadB10) -> A429_IN-
- J5 pad B11: unconnected-(J5-PadB11) -> A429_IN+
- J5 pad B12: unconnected-(J5-PadB12) -> A429_OUT+
- J5 pad B13: unconnected-(J5-PadB13) -> A429_OUT-
- J5 pad B14: unconnected-(J5-PadB14) -> SIN1
- J5 pad B15: unconnected-(J5-PadB15) -> SIN2
- J5 pad B16: unconnected-(J5-PadB16) -> GND
- J5 pad B17: unconnected-(J5-PadB17) -> BPOW
- J5 pad B18: unconnected-(J5-PadB18) -> GND
- J5 pad B19: unconnected-(J5-PadB19) -> DSI1
- J5 pad B2: unconnected-(J5-PadB2) -> TD+IN
- J5 pad B20: unconnected-(J5-PadB20) -> DSI2
- J5 pad B21: unconnected-(J5-PadB21) -> DSI3
- J5 pad B22: unconnected-(J5-PadB22) -> DSI4
- J5 pad B23: unconnected-(J5-PadB23) -> DSI5
- J5 pad B24: unconnected-(J5-PadB24) -> DSI6
- J5 pad B25: unconnected-(J5-PadB25) -> GND
- J5 pad B26: unconnected-(J5-PadB26) -> GND
- J5 pad B27: unconnected-(J5-PadB27) -> DOFB1
- J5 pad B28: unconnected-(J5-PadB28) -> DOFB2
- J5 pad B29: unconnected-(J5-PadB29) -> DOFB3
- J5 pad B3: unconnected-(J5-PadB3) -> RTD-IN
- J5 pad B30: unconnected-(J5-PadB30) -> DOFB4
- J5 pad B31: unconnected-(J5-PadB31) -> DOFB5
- J5 pad B32: unconnected-(J5-PadB32) -> DOFB6
- J5 pad B4: unconnected-(J5-PadB4) -> RTD+IN
- J5 pad B5: unconnected-(J5-PadB5) -> DAC_OUT
- J5 pad B6: unconnected-(J5-PadB6) -> GND
- J5 pad B7: unconnected-(J5-PadB7) -> CANHI
- J5 pad B8: unconnected-(J5-PadB8) -> CANLO
- J5 pad B9: unconnected-(J5-PadB9) -> GND
Routing:
- net GND: track 411.0 -> 430.0 mm, vias 213 -> 219
- net A429_OUT+: track 285.3 -> 292.2 mm
- net TD+IN: track 307.4 -> 313.9 mm
- net SIN1: track 166.8 -> 173.3 mm
- net RTD+IN: track 295.7 -> 302.2 mm
- net DSI6: track 94.5 -> 101.0 mm
- net DSI4: track 120.8 -> 127.3 mm
- net DSI2: track 134.4 -> 140.9 mm
- net DOFB6: track 91.1 -> 97.6 mm
- net DOFB4: track 114.7 -> 121.2 mm
- net DOFB2: track 143.2 -> 149.7 mm
- net CANLO: track 65.0 -> 71.5 mm
- net A429_IN-: track 288.8 -> 295.3 mm
- net TD-IN: track 200.1 -> 202.6 mm
- net SIN2: track 191.3 -> 193.8 mm
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
Commit message: Changed K to k on resistors
Parts:
- R38, R39, R40, R41, R42, R43, R44, R45, R46, R47, R48, R49: value 1K -> 1k
- R5, R55, R56, R57, R58, R59, R60: value 10K -> 10k
- R50, R51, R52, R53: value 100K -> 100k
Changed lines of the file:
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@@
 			)
 		)
-		(property "Value" "1K"
+		(property "Value" "1k"
 			(at 0 1.65 -90)
 			(layer "F.Fab")
@@
 			)
 		)
-		(property "Value" "1K"
+		(property "Value" "1k"
 			(at 0 1.65 -90)
 			(layer "F.Fab")
@@
 			)
 		)
-		(property "Value" "10K"
+		(property "Value" "10k"
 			(at 0 1.65 0)
 			(layer "F.Fab")
@@
 			)
 		)
-		(property "Value" "1K"
+		(property "Value" "1k"
 			(at 0 1.65 -90)
 			(layer "F.Fab")
@@
 			)
 		)
-		(property "Value" "10K"
+		(property "Value" "10k"
 			(at 0 1.65 -90)
 			(layer "F.Fab")
@@
 			)
 		)
-		(property "Value" "1K"
+		(property "Value" "1k"
 			(at 0 1.65 0)
 			(layer "F.Fab")
@@
 			)
 		)
-		(property "Value" "1K"
+		(property "Value" "1k"
 			(at 0 1.65 -90)
 			(layer "F.Fab")
@@
 			)
 		)
-		(property "Value" "10K"
+		(property "Value" "10k"
 			(at 0 1.65 90)
 			(layer "F.Fab")
@@
 			)
 		)
-		(property "Value" "1K"
+		(property "Value" "1k"
 			(at 0 1.65 0)
 			(layer "F.Fab")
@@
 			)
 		)
-		(property "Value" "1K"
+		(property "Value" "1k"
 			(at 0 -1.65 0)
 			(layer "B.Fab")
@@
 			)
 		)
-		(property "Value" "100K"
+		(property "Value" "100k"
 			(at 0 -1.65 0)
 			(layer "B.Fab")
@@
 			)
 		)
-		(property "Value" "1K"
+		(property "Value" "1k"
 			(at 0 -1.65 -90)
 			(layer "B.Fab")
@@
 			)
 		)
-		(property "Value" "1K"
+		(property "Value" "1k"
 			(at 0 -1.65 0)
 			(layer "B.Fab")
@@
 			)
 		)
-		(property "Value" "1K"
+		(property "Value" "1k"
 			(at 0 -1.65 90)
 			(layer "B.Fab")
@@
 			)
 		)
-		(property "Value" "1K"
+		(property "Value" "1k"
 			(at 0 -1.65 -90)
 			(layer "B.Fab")
@@
 			)
 		)
-		(property "Value" "10K"
+		(property "Value" "10k"
 			(at 0 -1.65 90)
 			(layer "B.Fab")
@@
 			)
 		)
-		(property "Value" "100K"
+		(property "Value" "100k"
 			(at 0 -1.65 -90)
 			(layer "B.Fab")
@@
 			)
 		)
-		(property "Value" "1K"
+		(property "Value" "1k"
 			(at 0 -1.65 -90)
 			(layer "B.Fab")
@@
 			)
 		)
-		(property "Value" "100K"
+		(property "Value" "100k"
 			(at 0 -1.65 -90)
 			(layer "B.Fab")
@@
 			)
 		)
-		(property "Value" "10K"
+		(property "Value" "10k"
 			(at 0 -1.65 -90)
 			(layer "B.Fab")
@@
 			)
 		)
-		(property "Value" "10K"
+		(property "Value" "10k"
 			(at 0 -1.65 -90)
 			(layer "B.Fab")
@@
 			)
 		)
-		(property "Value" "10K"
+		(property "Value" "10k"
 			(at 0 -1.65 90)
 			(layer "B.Fab")
@@
 			)
 		)
-		(property "Value" "100K"
+		(property "Value" "100k"
 			(at 0 -1.65 0)
 			(layer "B.Fab")

Commit message: Generated PCB BOM & CSV
Parts:
- R54: value 100K -> 100k
Changed lines of the file:
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@@
 			(disableapertmacros no)
 			(usegerberextensions yes)
-			(usegerberattributes no)
+			(usegerberattributes yes)
 			(usegerberadvancedattributes no)
 			(creategerberjobfile no)
@@
 			(viasonmask no)
 			(mode 1)
-			(useauxorigin no)
+			(useauxorigin yes)
 			(hpglpennumber 1)
 			(hpglpenspeed 20)
@@
 			(plotinvisibletext no)
 			(sketchpadsonfab no)
-			(subtractmaskfromsilk yes)
+			(subtractmaskfromsilk no)
 			(outputformat 1)
 			(mirror no)
 			(drillshape 0)
 			(scaleselection 1)
-			(outputdirectory "Backplane-backups/")
+			(outputdirectory "Files for Production/Gerber/")
 		)
 	)
@@
 			)
 		)
-		(property "Value" "100K"
+		(property "Value" "100k"
 			(at 0 -1.65 180)
 			(layer "B.Fab")
